Commit message: First revised commit

File: urdf/rrr_arm.urdf (robot description, URDF)
Before this commit: robot rpr_arm, 7 links, 6 joints
Links:
- link base_link: geometry collision mesh filename=package://rrr_arm/meshes/base_link.STL; visual mesh filename=package://rrr_arm/meshes/base_link.STL
- link gripper_left: geometry collision mesh filename=package://rrr_arm/meshes/gripper_left.STL; visual mesh filename=package://rrr_arm/meshes/gripper_left.STL
- link gripper_right: geometry collision mesh filename=package://rrr_arm/meshes/gripper_right.STL; visual mesh filename=package://rrr_arm/meshes/gripper_right.STL
- link link_1: geometry collision mesh filename=package://rrr_arm/meshes/link_1.STL; visual mesh filename=package://rrr_arm/meshes/link_1.STL
- link link_2: geometry collision mesh filename=package://rrr_arm/meshes/link_2.STL; visual mesh filename=package://rrr_arm/meshes/link_2.STL
- link link_3: geometry collision mesh filename=package://rrr_arm/meshes/link_3.STL; visual mesh filename=package://rrr_arm/meshes/link_3.STL
